Commit message: FIX: collision model for top structure depends on dual/single

File: fr3_husky_description/robots/husky_base.xacro (robot description, xacro)
@@ -69,13 +69,15 @@
         <origin rpy="0 0 0" xyz="0 0 0.006"/>
         <geometry>
-          <box size="0.85 0.65 0.012"/>
+          <box size="0.90 0.65 0.012"/>
         </geometry>
       </collision>
-      <collision>
-        <origin rpy="0 0 0" xyz="0.32 0 0.018"/>
-        <geometry>
-          <box size="0.25 0.35 0.01"/>
-        </geometry>
-      </collision>
+      <xacro:if value="${single_mani}">
+          <collision>
+            <origin rpy="0 0 0" xyz="0.32 0 0.018"/>
+            <geometry>
+              <box size="0.25 0.35 0.01"/>
+            </geometry>
+          </collision>
+      </xacro:if>
       <collision>
         <origin rpy="0 0 0" xyz="-0.28 0 0.65"/>
