Commit message: Modification: for index of urdf link, change joint name

File: fr3_husky_description/robots/dual_fr3_husky.urdf.xacro (robot description, xacro)
@@ -99,5 +99,5 @@
         <origin rpy="0 0 0" xyz="0 0 0.248"/>
     </joint>
-    <joint name="tmp_base_joint" type="fixed">
+    <joint name="base_joint" type="fixed">
         <parent link="base_link"/>
         <child link="tmp_base"/>
