Commit message: FIX: parameters

File: fr3_husky_description/robots/dual_fr3.srdf.xacro (robot description, xacro)
@@ -9,5 +9,5 @@
     <xacro:arg name="mobile" default="false"/>
     <!-- Should self-collision be enabled? -->
-    <xacro:arg name="with_sc" default="true" />
+    <xacro:arg name="with_sc" default="false" />
     <!-- ============================================================= -->
     <xacro:franka_arm_srdf arm_id="fr3"

File: fr3_husky_description/robots/single_fr3.srdf.xacro (robot description, xacro)
@@ -4,11 +4,11 @@
     <!-- ============================================================= -->
     <!-- Which arm: left or right -->
-    <xacro:arg name="side" default=""/>
+    <xacro:arg name="side" default="left"/>
     <!-- Should an end-effector be mounted at the flange? -->
     <xacro:arg name="hand" default="true" />
     <!-- Is base husky or just box-shaped? -->
-    <xacro:arg name="mobile" default="true"/>
+    <xacro:arg name="mobile" default="false"/>
     <!-- Should self-collision be enabled? -->
-    <xacro:arg name="with_sc" default="true" />
+    <xacro:arg name="with_sc" default="false" />
     <!-- ============================================================= -->
     <!-- Derived arm_prefix from side -->

File: fr3_husky_description/robots/single_fr3.urdf.xacro (robot description, xacro)
@@ -7,9 +7,9 @@
     <!-- ============================================================= -->
     <!-- Which arm: left or right -->
-    <xacro:arg name="side" default=""/>
+    <xacro:arg name="side" default="left"/>
     <!-- Should an end-effector be mounted at the flange? -->
     <xacro:arg name="hand" default="true" />
     <!-- Should self-collision be enabled? -->
-    <xacro:arg name="with_sc" default="true" />
+    <xacro:arg name="with_sc" default="false" />
     <!-- Is the robot being controlled with ros2_control?" -->
     <xacro:arg name="ros2_control" default="false" />
@@ -19,7 +19,7 @@
     <xacro:arg name="fake_sensor_commands" default="false" />
     <!-- Is base husky or just box-shaped? -->
-    <xacro:arg name="mobile" default="true"/>
+    <xacro:arg name="mobile" default="false"/>
     <!-- Use franka hand finger joint as fixed? -->
-    <xacro:arg name="fix_finger" default="true"/>
+    <xacro:arg name="fix_finger" default="false"/>
     <!-- ============================================================= -->
     <!-- Derived properties from side -->
@@ -29,7 +29,4 @@
     <xacro:property name="robot_ip"
                     value="${'172.16.5.5' if side_val == 'left' else '172.16.6.6'}"/>
-    <!-- prefix formatting (left_ / right_) -->
-    <xacro:property name="modified_prefix"
-                    value="${arm_prefix + '_' if arm_prefix else ''}"/>
     <!-- Base selection -->
     <xacro:unless value="$(arg mobile)">
@@ -61,5 +58,5 @@
                         gazebo_effort="false"
                         no_prefix="false"
-                        arm_prefix="${modified_prefix}"
+                        arm_prefix="${arm_prefix}"
                         description_pkg="franka_description"
                         connected_to="tmp_base"

Commit message: add: realsense

File: fr3_husky_description/robots/dual_fr3.srdf.xacro (robot description, xacro)
@@ -531,4 +531,6 @@
             <disable_collisions link1="left_fr3_hand_sc" link2="right_fr3_leftfinger" reason="User"/>
             <disable_collisions link1="left_fr3_hand_sc" link2="right_fr3_rightfinger" reason="User"/>
+            <!-- left hand sc - right hand sc -->
+            <disable_collisions link1="left_fr3_hand_sc" link2="right_fr3_hand_sc" reason="User"/>
             <!-- left hand - right link -->
             <disable_collisions link1="left_fr3_hand" link2="right_fr3_link0" reason="User"/>

File: fr3_husky_description/robots/dual_fr3.urdf.xacro (robot description, xacro)
@@ -2,4 +2,5 @@
 <robot xmlns:xacro="http://www.ros.org/wiki/xacro" name="fr3">
     <xacro:include filename="$(find franka_description)/robots/common/franka_multi_robot.xacro"/>
+    <xacro:include filename="$(find fr3_husky_description)/robots/realsense_d435i.urdf.xacro"/>
     <!-- base xacro includes -->
     <xacro:include filename="$(find fr3_husky_description)/robots/box_base.xacro"/>
@@ -55,4 +56,35 @@
         <origin rpy="0 0 0" xyz="0 0 0"/>
     </joint>
+    <!-- Load ee→camera TF calibration for each arm -->
+    <xacro:property name="ee2cam_tf_left"
+        value="${xacro.load_yaml('$(find fr3_husky_description)/config/TF_ee2cam_left.yaml')}"/>
+    <xacro:property name="ee2cam_tf_right"
+        value="${xacro.load_yaml('$(find fr3_husky_description)/config/TF_ee2cam_right.yaml')}"/>
+    <xacro:realsense_d435i is_reverse="true" prefix="left"/>
+    <xacro:realsense_d435i is_reverse="true" prefix="right"/>
+    <joint name="left_ee2d435i" type="fixed">
+        <xacro:if value="$(arg hand)">
+            <parent link="left_fr3_hand"/>
+        </xacro:if>
+        <xacro:unless value="$(arg hand)">
+            <parent link="left_fr3_link8"/>
+        </xacro:unless>
+        <child link="left_d435i_color_optical_frame"/>
+        <origin
+            xyz="${ee2cam_tf_left['translation'][0]} ${ee2cam_tf_left['translation'][1]} ${ee2cam_tf_left['translation'][2]}"
+            rpy="${ee2cam_tf_left['euler_zyx'][0]} ${ee2cam_tf_left['euler_zyx'][1]} ${ee2cam_tf_left['euler_zyx'][2]}"/>
+    </joint>
+    <joint name="right_ee2d435i" type="fixed">
+        <xacro:if value="$(arg hand)">
+            <parent link="right_fr3_hand"/>
+        </xacro:if>
+        <xacro:unless value="$(arg hand)">
+            <parent link="right_fr3_link8"/>
+        </xacro:unless>
+        <child link="right_d435i_color_optical_frame"/>
+        <origin
+            xyz="${ee2cam_tf_right['translation'][0]} ${ee2cam_tf_right['translation'][1]} ${ee2cam_tf_right['translation'][2]}"
+            rpy="${ee2cam_tf_right['euler_zyx'][0]} ${ee2cam_tf_right['euler_zyx'][1]} ${ee2cam_tf_right['euler_zyx'][2]}"/>
+    </joint>
     <xacro:franka_multi_robot
         arm_ids="${arm_ids_str}"

File: fr3_husky_description/robots/dual_fr3_husky.srdf.xacro (robot description, xacro)
@@ -534,4 +534,6 @@
             <disable_collisions link1="left_fr3_hand_sc" link2="right_fr3_leftfinger" reason="User"/>
             <disable_collisions link1="left_fr3_hand_sc" link2="right_fr3_rightfinger" reason="User"/>
+            <!-- left hand sc - right hand sc -->
+            <disable_collisions link1="left_fr3_hand_sc" link2="right_fr3_hand_sc" reason="User"/>
             <!-- left hand - right link -->
             <disable_collisions link1="left_fr3_hand" link2="right_fr3_link0" reason="User"/>

File: fr3_husky_description/robots/dual_fr3_husky.urdf.xacro (robot description, xacro)
@@ -3,4 +3,5 @@
     <xacro:include filename="$(find franka_description)/robots/common/franka_multi_robot.xacro"/>
     <xacro:include filename="$(find husky_description)/urdf/husky_macro.urdf.xacro" />
+    <xacro:include filename="$(find fr3_husky_description)/robots/realsense_d435i.urdf.xacro"/>
     <!-- ============================================================= -->
     <!-- Should an end-effector be mounted at the flange? -->
@@ -105,4 +106,35 @@
         <origin rpy="0 0 0" xyz="0 0 0"/>
     </joint>
+    <!-- Load ee→camera TF calibration for each arm -->
+    <xacro:property name="ee2cam_tf_left"
+        value="${xacro.load_yaml('$(find fr3_husky_description)/config/TF_ee2cam_left.yaml')}"/>
+    <xacro:property name="ee2cam_tf_right"
+        value="${xacro.load_yaml('$(find fr3_husky_description)/config/TF_ee2cam_right.yaml')}"/>
+    <xacro:realsense_d435i is_reverse="true" prefix="left"/>
+    <xacro:realsense_d435i is_reverse="true" prefix="right"/>
+    <joint name="left_ee2d435i" type="fixed">
+        <xacro:if value="$(arg hand)">
+            <parent link="left_fr3_hand"/>
+        </xacro:if>
+        <xacro:unless value="$(arg hand)">
+            <parent link="left_fr3_link8"/>
+        </xacro:unless>
+        <child link="left_d435i_color_optical_frame"/>
+        <origin
+            xyz="${ee2cam_tf_left['translation'][0]} ${ee2cam_tf_left['translation'][1]} ${ee2cam_tf_left['translation'][2]}"
+            rpy="${ee2cam_tf_left['euler_zyx'][0]} ${ee2cam_tf_left['euler_zyx'][1]} ${ee2cam_tf_left['euler_zyx'][2]}"/>
+    </joint>
+    <joint name="right_ee2d435i" type="fixed">
+        <xacro:if value="$(arg hand)">
+            <parent link="right_fr3_hand"/>
+        </xacro:if>
+        <xacro:unless value="$(arg hand)">
+            <parent link="right_fr3_link8"/>
+        </xacro:unless>
+        <child link="right_d435i_color_optical_frame"/>
+        <origin
+            xyz="${ee2cam_tf_right['translation'][0]} ${ee2cam_tf_right['translation'][1]} ${ee2cam_tf_right['translation'][2]}"
+            rpy="${ee2cam_tf_right['euler_zyx'][0]} ${ee2cam_tf_right['euler_zyx'][1]} ${ee2cam_tf_right['euler_zyx'][2]}"/>
+    </joint>
     <xacro:franka_multi_robot
         arm_ids="${arm_ids_str}"

File: fr3_husky_description/robots/single_fr3.urdf.xacro (robot description, xacro)
@@ -5,4 +5,5 @@
     <xacro:include filename="$(find fr3_husky_description)/robots/box_base.xacro"/>
     <xacro:include filename="$(find fr3_husky_description)/robots/husky_base.xacro"/>
+    <xacro:include filename="$(find fr3_husky_description)/robots/realsense_d435i.urdf.xacro"/>
     <!-- ============================================================= -->
     <!-- Which arm: left or right -->
@@ -70,3 +71,19 @@
         <origin rpy="0 0 0" xyz="0 0 0"/>
     </joint>
+    <!-- Load ee->camera TF calibration depending on which arm side -->
+    <xacro:property name="ee2cam_tf"
+        value="${xacro.load_yaml('$(find fr3_husky_description)/config/TF_ee2cam_$(arg side).yaml')}"/>
+    <xacro:realsense_d435i is_reverse="true" prefix="${arm_prefix}"/>
+    <joint name="${arm_prefix}_ee2d435i" type="fixed">
+        <xacro:if value="$(arg hand)">
+            <parent link="${arm_prefix}_fr3_hand"/>
+        </xacro:if>
+        <xacro:unless value="$(arg hand)">
+            <parent link="${arm_prefix}_fr3_link8"/>
+        </xacro:unless>
+        <child link="${arm_prefix}_d435i_color_optical_frame"/>
+        <origin
+            xyz="${ee2cam_tf['translation'][0]} ${ee2cam_tf['translation'][1]} ${ee2cam_tf['translation'][2]}"
+            rpy="${ee2cam_tf['euler_zyx'][0]} ${ee2cam_tf['euler_zyx'][1]} ${ee2cam_tf['euler_zyx'][2]}"/>
+    </joint>
 </robot>

File: fr3_husky_description/robots/single_fr3_husky.urdf.xacro (robot description, xacro)
@@ -3,4 +3,5 @@
     <xacro:include filename="$(find franka_description)/robots/common/franka_robot.xacro"/>
     <xacro:include filename="$(find husky_description)/urdf/husky_macro.urdf.xacro" />
+    <xacro:include filename="$(find fr3_husky_description)/robots/realsense_d435i.urdf.xacro"/>
     <!-- ============================================================= -->
     <!-- Which arm: left or right -->
@@ -138,3 +139,19 @@
         <origin rpy="0 0 0" xyz="0.36 0.0 0.27"/>
     </joint>
+    <!-- Load ee→camera TF calibration depending on which arm side -->
+    <xacro:property name="ee2cam_tf"
+        value="${xacro.load_yaml('$(find fr3_husky_description)/config/TF_ee2cam_$(arg side).yaml')}"/>
+    <xacro:realsense_d435i is_reverse="true" prefix="${arm_prefix}"/>
+    <joint name="${arm_prefix}_ee2d435i" type="fixed">
+        <xacro:if value="$(arg hand)">
+            <parent link="${arm_prefix}_fr3_hand"/>
+        </xacro:if>
+        <xacro:unless value="$(arg hand)">
+            <parent link="${arm_prefix}_fr3_link8"/>
+        </xacro:unless>
+        <child link="${arm_prefix}_d435i_color_optical_frame"/>
+        <origin
+            xyz="${ee2cam_tf['translation'][0]} ${ee2cam_tf['translation'][1]} ${ee2cam_tf['translation'][2]}"
+            rpy="${ee2cam_tf['euler_zyx'][0]} ${ee2cam_tf['euler_zyx'][1]} ${ee2cam_tf['euler_zyx'][2]}"/>
+    </joint>
 </robot>
