Commit message: add: azure kinect

File: fr3_husky_description/robots/dual_fr3.urdf.xacro (robot description, xacro)
@@ -3,4 +3,5 @@
     <xacro:include filename="$(find franka_description)/robots/common/franka_multi_robot.xacro"/>
     <xacro:include filename="$(find fr3_husky_description)/robots/realsense_d435i.urdf.xacro"/>
+    <xacro:include filename="$(find fr3_husky_description)/robots/azure_kinect.urdf.xacro"/>
     <!-- base xacro includes -->
     <xacro:include filename="$(find fr3_husky_description)/robots/box_base.xacro"/>
@@ -56,4 +57,16 @@
         <origin rpy="0 0 0" xyz="0 0 0"/>
     </joint>
+    <xacro:if value="$(arg mobile)">
+        <!-- Load base->camera TF calibration -->
+        <xacro:property name="base2cam_tf"  value="${xacro.load_yaml('$(find fr3_husky_description)/config/TF_base2cam.yaml')}"/>
+        <xacro:azure_kinect is_reverse="true" prefix="top"/>
+        <joint name="base2top_cam" type="fixed">
+            <parent link="mobile_base"/>
+            <child link="top_azure_rgb_link"/>
+            <origin
+                xyz="${base2cam_tf['translation'][0]} ${base2cam_tf['translation'][1]} ${base2cam_tf['translation'][2]}"
+                rpy="${base2cam_tf['euler_zyx'][0]}   ${base2cam_tf['euler_zyx'][1]}   ${base2cam_tf['euler_zyx'][2]}"/>
+        </joint>
+    </xacro:if>
     <!-- Load ee→camera TF calibration for each arm -->
     <xacro:property name="ee2cam_tf_left"

File: fr3_husky_description/robots/dual_fr3_husky.urdf.xacro (robot description, xacro)
@@ -4,4 +4,5 @@
     <xacro:include filename="$(find husky_description)/urdf/husky_macro.urdf.xacro" />
     <xacro:include filename="$(find fr3_husky_description)/robots/realsense_d435i.urdf.xacro"/>
+    <xacro:include filename="$(find fr3_husky_description)/robots/azure_kinect.urdf.xacro"/>
     <!-- ============================================================= -->
     <!-- Should an end-effector be mounted at the flange? -->
@@ -106,4 +107,14 @@
         <origin rpy="0 0 0" xyz="0 0 0"/>
     </joint>
+    <!-- Load base->camera TF calibration -->
+    <xacro:property name="base2cam_tf"  value="${xacro.load_yaml('$(find fr3_husky_description)/config/TF_base2cam.yaml')}"/>
+    <xacro:azure_kinect is_reverse="true" prefix="top"/>
+    <joint name="base2top_cam" type="fixed">
+        <parent link="base_link"/>
+        <child link="top_azure_rgb_link"/>
+        <origin
+            xyz="${base2cam_tf['translation'][0]} ${base2cam_tf['translation'][1]} ${base2cam_tf['translation'][2]}"
+            rpy="${base2cam_tf['euler_zyx'][0]}   ${base2cam_tf['euler_zyx'][1]}   ${base2cam_tf['euler_zyx'][2]}"/>
+    </joint>
     <!-- Load ee→camera TF calibration for each arm -->
     <xacro:property name="ee2cam_tf_left"

File: fr3_husky_description/robots/single_fr3.urdf.xacro (robot description, xacro)
@@ -6,4 +6,5 @@
     <xacro:include filename="$(find fr3_husky_description)/robots/husky_base.xacro"/>
     <xacro:include filename="$(find fr3_husky_description)/robots/realsense_d435i.urdf.xacro"/>
+    <xacro:include filename="$(find fr3_husky_description)/robots/azure_kinect.urdf.xacro"/>
     <!-- ============================================================= -->
     <!-- Which arm: left or right -->
@@ -71,4 +72,16 @@
         <origin rpy="0 0 0" xyz="0 0 0"/>
     </joint>
+    <xacro:if value="$(arg mobile)">
+        <!-- Load base->camera TF calibration -->
+        <xacro:property name="base2cam_tf"  value="${xacro.load_yaml('$(find fr3_husky_description)/config/TF_base2cam.yaml')}"/>
+        <xacro:azure_kinect is_reverse="true" prefix="top"/>
+        <joint name="base2top_cam" type="fixed">
+            <parent link="mobile_base"/>
+            <child link="top_azure_rgb_link"/>
+            <origin
+                xyz="${base2cam_tf['translation'][0]} ${base2cam_tf['translation'][1]} ${base2cam_tf['translation'][2]}"
+                rpy="${base2cam_tf['euler_zyx'][0]}   ${base2cam_tf['euler_zyx'][1]}   ${base2cam_tf['euler_zyx'][2]}"/>
+        </joint>
+    </xacro:if>
     <!-- Load ee->camera TF calibration depending on which arm side -->
     <xacro:property name="ee2cam_tf"

File: fr3_husky_description/robots/single_fr3_husky.urdf.xacro (robot description, xacro)
@@ -4,4 +4,5 @@
     <xacro:include filename="$(find husky_description)/urdf/husky_macro.urdf.xacro" />
     <xacro:include filename="$(find fr3_husky_description)/robots/realsense_d435i.urdf.xacro"/>
+    <xacro:include filename="$(find fr3_husky_description)/robots/azure_kinect.urdf.xacro"/>
     <!-- ============================================================= -->
     <!-- Which arm: left or right -->
@@ -139,4 +140,14 @@
         <origin rpy="0 0 0" xyz="0.36 0.0 0.27"/>
     </joint>
+    <!-- Load base->camera TF calibration -->
+    <xacro:property name="base2cam_tf"  value="${xacro.load_yaml('$(find fr3_husky_description)/config/TF_base2cam.yaml')}"/>
+    <xacro:azure_kinect is_reverse="true" prefix="top"/>
+    <joint name="base2top_cam" type="fixed">
+        <parent link="base_link"/>
+        <child link="top_azure_rgb_link"/>
+        <origin
+            xyz="${base2cam_tf['translation'][0]} ${base2cam_tf['translation'][1]} ${base2cam_tf['translation'][2]}"
+            rpy="${base2cam_tf['euler_zyx'][0]}   ${base2cam_tf['euler_zyx'][1]}   ${base2cam_tf['euler_zyx'][2]}"/>
+    </joint>
     <!-- Load ee→camera TF calibration depending on which arm side -->
     <xacro:property name="ee2cam_tf"
